File: PresensePCB/PresensePCB.kicad_sch (KiCad schematic)
At the start: 3 parts, among them U1 ESP32-C3_SUPERMINI_TH, U2 VEML7700, U3 LD2420

Commit message: pcb design complete
Parts:
- removed U3: LD2420, LD2420:LD2420_Module, symbol LD2420:LD2420
- added D1, D2, D3, D4, D5: WS2812B-2020, LED_SMD:LED_WS2812B-2020_PLCC4_2.0x2.0mm, symbol LED:WS2812B-2020
- added LD2420: LD2420_Module, LD2420:LD2420_Module, symbol LD2420:LD2420_Module
- added R_OUT1: 0R, Resistor_SMD:R_0805_2012Metric_Pad1.20x1.40mm_HandSolder, symbol Device:R_Small
- added TP223B1: TP223B, TP223B:TP223B_Module, symbol TP223B:TP223B_Module
- renumbered U1 to ESP32C3, U2 to VEML7700
Connections:
- net +5V: now reaches VEML7700.1 (VCC)
- net +5V: now also ESP32C3.5V, D1.4 (VDD), D2.4 (VDD), D3.4 (VDD), D4.4 (VDD), D5.4 (VDD), LD2420.1 (VCC)
- net GND: now reaches VEML7700.3 (GND)
- net GND: now also ESP32C3.G (GND), D1.2 (VSS), D2.2 (VSS), D3.2 (VSS), D4.2 (VSS), D5.2 (VSS), LD2420.2 (GND), TP223B1.3 (GND)
- net G9: now reaches VEML7700.4 (SCL)
- net G9: now also ESP32C3.9 (GPIO9)
- net G8: now reaches VEML7700.5 (SDA)
- net G8: now also ESP32C3.8 (GPIO8)
- net G3: now reaches ESP32C3.3 (GPIO3)
- net G3: now also TP223B1.2 (OUT)
- net +3.3V: now reaches ESP32C3.3.3 (3V3)
- net +3.3V: now also TP223B1.1 (VCC)
- net G4: now reaches ESP32C3.4 (GPIO4)
- net G4: now also LD2420.4 (RX)
- net G5: now reaches ESP32C3.5 (GPIO5)
- net G5: now also LD2420.3 (TX)
- net G6: now reaches ESP32C3.6 (GPIO6)
- net G6: now also D1.3 (DIN)
- net G7: now reaches ESP32C3.7 (GPIO7)
- net G7: now also R_OUT1.2
- new net: D4.1 (DOUT), D5.3 (DIN)
- new net: D3.1 (DOUT), D4.3 (DIN)
- new net: D1.1 (DOUT), D2.3 (DIN)
- new net: D2.1 (DOUT), D3.3 (DIN)
- new net: LD2420.5 (OUT), R_OUT1.1
