File: PresensePCB/PresensePCB.kicad_pcb (KiCad board)
At the start: 2 copper layers, 22 x 78.5 mm, 10 parts

Commit message: generate pcb
Other:
- board text added: "JLCJLCJLCJLC"
- board text added: "Presence 1 Madhukar Temba Rev 2026-02-02"
